Commit message: GZ対応

File: src/piper_description/urdf/piper_description_gazebo.xacro (robot description, xacro)
@@ -3,4 +3,6 @@
   name="piper"
   xmlns:xacro="http://ros.org/wiki/xacro">
+  <xacro:arg name="use_gz" default="true"/>
+  <xacro:property name="use_gz" value="$(arg use_gz)"/>
 <!-- world -->
   <link name="world"/>
@@ -397,10 +399,10 @@
         value="0.025" />
       <inertia
-        ixx="0.00007371"
-        ixy="-0.00000113"
-        ixz="0.00000021"
-        iyy="-0.00000113"
-        iyz="-0.00001372"
-        izz="0.0000747" />
+        ixx="0.000075"
+        ixy="0.0"
+        ixz="0.0"
+        iyy="0.000075"
+        iyz="0.0"
+        izz="0.000075" />
     </inertial>
     <visual>
@@ -455,10 +457,10 @@
         value="0.025" />
       <inertia
-        ixx="0.00007371"
-        ixy="-0.00000113"
-        ixz="0.00000021"
-        iyy="-0.00000113"
-        iyz="-0.00001372"
-        izz="0.0000747" />
+        ixx="0.000075"
+        ixy="0.0"
+        ixz="0.0"
+        iyy="0.000075"
+        iyz="0.0"
+        izz="0.000075" />
     </inertial>
     <visual>
@@ -537,5 +539,10 @@
   <ros2_control name="GazeboSystem" type="system">
       <hardware>
-          <plugin>gazebo_ros2_control/GazeboSystem</plugin>
+          <xacro:if value="${use_gz}">
+              <plugin>gz_ros2_control/GazeboSimSystem</plugin>
+          </xacro:if>
+          <xacro:unless value="${use_gz}">
+              <plugin>gazebo_ros2_control/GazeboSystem</plugin>
+          </xacro:unless>
       </hardware>
       <joint name="joint1">
@@ -620,10 +627,20 @@
       </joint>
   </ros2_control>
-<!-- gazebo -->
-  <gazebo>
-    <plugin name="gazebo_ros2_control" filename="libgazebo_ros2_control.so">
-        <parameters> $(find piper_gazebo)/config/ros2_controllers.yaml </parameters>
-        <robot_param_node>robot_state_publisher</robot_param_node>
-    </plugin>
-  </gazebo>
+<!-- gazebo / gz -->
+  <xacro:if value="${use_gz}">
+    <gazebo>
+      <plugin name="gz_ros2_control::GazeboSimROS2ControlPlugin" filename="libgz_ros2_control-system.so">
+          <parameters> $(find piper_gazebo)/config/ros2_controllers.yaml </parameters>
+          <robot_param>robot_description</robot_param>
+      </plugin>
+    </gazebo>
+  </xacro:if>
+  <xacro:unless value="${use_gz}">
+    <gazebo>
+      <plugin name="gazebo_ros2_control" filename="libgazebo_ros2_control.so">
+          <parameters> $(find piper_gazebo)/config/ros2_controllers.yaml </parameters>
+          <robot_param_node>robot_state_publisher</robot_param_node>
+      </plugin>
+    </gazebo>
+  </xacro:unless>
 </robot>

File: src/piper_description/urdf/piper_no_gripper_description_gazebo.xacro (robot description, xacro)
@@ -3,4 +3,6 @@
   name="piper"
   xmlns:xacro="http://ros.org/wiki/xacro">
+  <xacro:arg name="use_gz" default="true"/>
+  <xacro:property name="use_gz" value="$(arg use_gz)"/>
 <!-- world -->
   <link name="world"/>
@@ -364,5 +366,10 @@
   <ros2_control name="GazeboSystem" type="system">
       <hardware>
-          <plugin>gazebo_ros2_control/GazeboSystem</plugin>
+          <xacro:if value="${use_gz}">
+              <plugin>gz_ros2_control/GazeboSimSystem</plugin>
+          </xacro:if>
+          <xacro:unless value="${use_gz}">
+              <plugin>gazebo_ros2_control/GazeboSystem</plugin>
+          </xacro:unless>
       </hardware>
       <joint name="joint1">
@@ -427,10 +434,20 @@
       </joint>
   </ros2_control>
-<!-- gazebo -->
-  <gazebo>
-    <plugin name="gazebo_ros2_control" filename="libgazebo_ros2_control.so">
-        <parameters> $(find piper_gazebo)/config/ros2_no_gripper_controllers.yaml </parameters>
-        <robot_param_node>robot_state_publisher</robot_param_node>
-    </plugin>
-  </gazebo>
+<!-- gazebo / gz -->
+  <xacro:if value="${use_gz}">
+    <gazebo>
+      <plugin name="gz_ros2_control::GazeboSimROS2ControlPlugin" filename="libgz_ros2_control-system.so">
+          <parameters> $(find piper_gazebo)/config/ros2_no_gripper_controllers.yaml </parameters>
+          <robot_param>robot_description</robot_param>
+      </plugin>
+    </gazebo>
+  </xacro:if>
+  <xacro:unless value="${use_gz}">
+    <gazebo>
+      <plugin name="gazebo_ros2_control" filename="libgazebo_ros2_control.so">
+          <parameters> $(find piper_gazebo)/config/ros2_no_gripper_controllers.yaml </parameters>
+          <robot_param_node>robot_state_publisher</robot_param_node>
+      </plugin>
+    </gazebo>
+  </xacro:unless>
 </robot>
